File: treeleafRelay.kicad_sch (KiCad schematic)
At the start: 0 parts

Commit message: Added esp
Parts:
- added U1: (no value), krafters-lib:esp32-s3-cam-devkit, symbol krafters_lib:esp32-s3_cam_devkit
Changed lines of the file:
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@@
 	(generator_version "10.0")
 	(paper "A4")
+	(symbol
+		(lib_id "krafters_lib:esp32-s3_cam_devkit")
+		(at 160.02 27.94 0)
+		(unit 1)
+		(body_style 1)
+		(exclude_from_sim no)
+		(in_bom yes)
+		(on_board yes)
+		(in_pos_files yes)
+		(dnp no)
+		(fields_autoplaced yes)
+		(property "Reference" "U1"
+			(at 172.085 26.67 0)
+			(show_name no)
+			(do_not_autoplace no)
+			(effects
+				(font
+					(size 1.27 1.27)
+				)
+			)
+		)
+		(property "Value" ""
+			(at 160.02 27.94 0)
+			(show_name no)
+			(do_not_autoplace no)
+			(effects
+				(font
+					(size 1.27 1.27)
+				)
+			)
+		)
+		(property "Footprint" "krafters-lib:esp32-s3-cam-devkit"
+			(at 160.02 27.94 0)
+			(hide yes)
+			(show_name no)
+			(do_not_autoplace no)
+			(effects
+				(font
+					(size 1.27 1.27)
+				)
+			)
+		)
+		(property "Datasheet" ""
+			(at 160.02 27.94 0)
+			(hide yes)
+			(show_name no)
+			(do_not_autoplace no)
+			(effects
+				(font
+					(size 1.27 1.27)
+				)
+			)
+		)
+		(property "Description" ""
+			(at 160.02 27.94 0)
+			(hide yes)
+			(show_name no)
+			(do_not_autoplace no)
+			(effects
+				(font
+					(size 1.27 1.27)
+				)
+			)
+		)
+		(pin "20"
+		)
+		(pin "10"
+		)
+		(pin "3"
+		)
+		(pin "15"
+		)
+		(pin "32"
+		)
+		(pin "9"
+		)
+		(pin "22"
+		)
+		(pin "29"
+		)
+		(pin "34"
+		)
+		(pin "12"
+		)
+		(pin "31"
+		)
+		(pin "26"
+		)
+		(pin "13"
+		)
+		(pin "16"
+		)
+		(pin "25"
+		)
+		(pin "37"
+		)
+		(pin "28"
+		)
+		(pin "23"
+		)
+		(pin "5"
+		)
+		(pin "2"
+		)
+		(pin "35"
+		)
+		(pin "1"
+		)
+		(pin "30"
+		)
+		(pin "40"
+		)
+		(pin "38"
+		)
+		(pin "6"
+		)
+		(pin "18"
+		)
+		(pin "24"
+		)
+		(pin "11"
+		)
+		(pin "39"
+		)
+		(pin "33"
+		)
+		(pin "8"
+		)
+		(pin "17"
+		)
+		(pin "27"
+		)
+		(pin "4"
+		)
+		(pin "14"
+		)
+		(pin "21"
+		)
+		(pin "19"
+		)
+		(pin "36"
+		)
+		(pin "7"
+		)
+		(instances
+			(project "treeleafRelay"
+				(path "/53fc10da-4791-471f-a9ac-5eadf28e4e6f"
+					(reference "U1")
+					(unit 1)
+				)
+			)
+		)
+	)
 	(sheet_instances
 		(path "/"
