File: cam_relay_device.kicad_sch (KiCad schematic)
At the start: 12 parts, among them K1 SRD-05VDC-SL-C, Q1 MMBT3904, U5 DB301V-3_5-2P-GN

Commit message: review and optmize for fab
Parts:
- added H1, H2, H3: MountingScrew, MountingHole:MountingHole_2.2mm_M2, symbol Auxiliary_Items:MountingScrew
- D1: footprint krafters-lib:SOD-123FL_L2.8-W1.8-LS3.7-RD -> krafters_lib_fp:SOD-123FL_L2.8-W1.8-LS3.7-RD
- K1: footprint krafters-lib:RELAY-TH_SRD-XXVDC-XL-C -> krafters_lib_fp:RELAY-TH_SRD-XXVDC-XL-C
- R1, R2, R3, R4, R5: footprint Resistor_SMD:R_0603_1608Metric -> krafters_lib_fp:R0603
- U1: footprint krafters-lib:esp32-s3-cam-devkit -> krafters_lib_fp:esp32-s3-cam-devkit
